Commit message: Add bundled robot models and test fixtures

File: robot_models/unitree_g1/g1_29dof_popsicle.urdf (robot description, URDF)
Before this commit: robot g1, 41 links, 40 joints
Links:
- link head_link: geometry visual mesh filename=meshes/head_link.STL
- link left_ankle_pitch_link: geometry visual mesh filename=meshes/left_ankle_pitch_link.STL
- link left_ankle_roll_link: geometry collision cylinder length=0.05 radius=0.01; collision cylinder length=0.05 radius=0.01
- link left_elbow_link: geometry collision cylinder length=0.13 radius=0.035; visual mesh filename=meshes/left_elbow_link.STL
- link left_hip_pitch_link: geometry visual mesh filename=meshes/left_hip_pitch_link.STL
- link left_hip_roll_link: geometry collision cylinder length=0.2 radius=0.05; visual mesh filename=meshes/left_hip_roll_link.STL
- link left_hip_yaw_link: geometry visual mesh filename=meshes/left_hip_yaw_link.STL
- link left_knee_link: geometry collision cylinder length=0.2 radius=0.05; visual mesh filename=meshes/left_knee_link.STL
- link left_rubber_hand: geometry visual mesh filename=meshes/left_rubber_hand.STL
- link left_shoulder_pitch_link: geometry visual mesh filename=meshes/left_shoulder_pitch_link.STL
- link left_shoulder_roll_link: geometry visual mesh filename=meshes/left_shoulder_roll_link.STL
- link left_shoulder_yaw_link: geometry collision cylinder length=0.13 radius=0.035; visual mesh filename=meshes/left_shoulder_yaw_link.STL
- link left_wrist_pitch_link: geometry visual mesh filename=meshes/left_wrist_pitch_link.STL
- link left_wrist_roll_link: geometry visual mesh filename=meshes/left_wrist_roll_link.STL
- link left_wrist_yaw_link: geometry collision cylinder length=0.05 radius=0.05; visual mesh filename=meshes/left_wrist_yaw_link.STL
- link logo_link: geometry visual mesh filename=meshes/logo_link.STL
- link pelvis: geometry collision sphere radius=0.07; visual mesh filename=meshes/pelvis.STL
- link pelvis_contour_link: geometry visual mesh filename=meshes/pelvis_contour_link.STL
- link right_ankle_pitch_link: geometry visual mesh filename=meshes/right_ankle_pitch_link.STL
- link right_ankle_roll_link: geometry collision cylinder length=0.05 radius=0.01; collision cylinder length=0.05 radius=0.01
- link right_elbow_link: geometry collision cylinder length=0.13 radius=0.035; visual mesh filename=meshes/right_elbow_link.STL
- link right_hip_pitch_link: geometry visual mesh filename=meshes/right_hip_pitch_link.STL
- link right_hip_roll_link: geometry collision cylinder length=0.2 radius=0.05; visual mesh filename=meshes/right_hip_roll_link.STL
- link right_hip_yaw_link: geometry visual mesh filename=meshes/right_hip_yaw_link.STL
- link right_knee_link: geometry collision cylinder length=0.2 radius=0.05; visual mesh filename=meshes/right_knee_link.STL
- link right_rubber_hand: geometry visual mesh filename=meshes/right_rubber_hand.STL
- link right_shoulder_pitch_link: geometry visual mesh filename=meshes/right_shoulder_pitch_link.STL
- link right_shoulder_roll_link: geometry visual mesh filename=meshes/right_shoulder_roll_link.STL
- link right_shoulder_yaw_link: geometry collision cylinder length=0.13 radius=0.035; visual mesh filename=meshes/right_shoulder_yaw_link.STL
- link right_wrist_pitch_link: geometry visual mesh filename=meshes/right_wrist_pitch_link.STL
- link right_wrist_roll_link: geometry visual mesh filename=meshes/right_wrist_roll_link.STL
- link right_wrist_yaw_link: geometry collision cylinder length=0.05 radius=0.05; visual mesh filename=meshes/right_wrist_yaw_link.STL
- link torso_link: geometry collision cylinder length=0.01 radius=0.068; collision cylinder length=0.04 radius=0.065
- link waist_roll_link: geometry visual mesh filename=meshes/waist_roll_link_rev_1_0.STL
- link waist_yaw_link: geometry visual mesh filename=meshes/waist_yaw_link_rev_1_0.STL
